File: hardware/sound-20d01mb/oscillators.sch (KiCad schematic (older format))
At the start: 0 parts

Commit message: Added OSC
Parts:
- added C? (x6): 0.1uF, Capacitor_SMD:C_1206_3216Metric_Pad1.42x1.75mm_HandSolder, symbol Device:C
- added D? (x2): LED, LED_SMD:LED_1206_3216Metric_Pad1.42x1.75mm_HandSolder, symbol Device:LED
- added R? (x2): 680R, Resistor_SMD:R_1206_3216Metric_Pad1.42x1.75mm_HandSolder, symbol Device:R
- added R? (x4): 51R, Resistor_SMD:R_1206_3216Metric_Pad1.42x1.75mm_HandSolder, symbol Device:R
- added R?: 10K, Resistor_SMD:R_1206_3216Metric_Pad1.42x1.75mm_HandSolder, symbol Device:R
- added U? (x2): 74LVC1G125, Package_TO_SOT_SMD:SOT-23-5_HandSoldering, symbol 74xGxx:74LVC1G125
- added U? (x2): 74LVC1G86, Package_TO_SOT_SMD:SOT-23-5_HandSoldering, symbol 74xGxx:74LVC1G86
- added X? (x2): DFA-S2, Oscillator:Oscillator_SMD_Fordahl_DFAS2-4Pin_7.3x5.1mm_HandSoldering, symbol Oscillator:DFA-S2
Connections:
- net OSC_OUTPUT: now also R?.2, R?.2
- net OSC_SEL: now also R?.1, U?.1, U?.2
- new net: D?.2 (A), R?.2 (x2)
- new net: R?.2, U?.2 (x2)
- new net: R?.1, U?.4 (x2)
- new net: R?.1, X?.3 (OUT) (x2)
- new net +3V3: C?.1, C?.1, C?.1, C?.1, C?.1, C?.1, R?.1, R?.1, U?.1, U?.5 (VCC), U?.5 (VCC), U?.5 (VCC), U?.5 (VCC), X?.4 (V+), X?.4 (V+)
- new net GND: C?.2, C?.2, C?.2, C?.2, C?.2, C?.2, R?.2, U?.2, U?.3 (GND), U?.3 (GND), U?.3 (GND), U?.3 (GND), X?.2 (GND), X?.2 (GND)
- new net OSC0: D?.1 (K), U?.1, U?.4
- new net OSC1: D?.1 (K), U?.1, U?.4
- no-connect marks 0 -> 2
