File: hardware/sound-20d01mb/mcu.sch (KiCad schematic (older format))
At the start: 23 parts

Commit message: Updated schematic
Connections:
- net PA4_NSS: now reaches U?.20 (PA4)
- net PA5_SCK: now reaches U?.21 (PA5)
- net PA6_MISO: now reaches U?.22 (PA6)
- net PA7_MOSI: now reaches U?.23 (PA7)
- net ~SHUTDOWN: now reaches U?.24 (PC4)
- net MUTE: now reaches U?.25 (PC5)
- net PB0_SDIO_D1: now reaches U?.26 (PB0)
- net PB1_SDIO_D2: now reaches U?.27 (PB1)
- net PB2_SDIO_CK: now reaches U?.28 (PB2)
- net PC8_SDIO_D0: now reaches U?.39 (PC8)
- net PC11_SDIO_D3: now reaches U?.52 (PC11)
- net PD2_SDIO_CMD: now reaches U?.54 (PD2)
Other:
- moved on the sheet: C?, R?
