File: hardware/sound-20d01mb/dac.sch (KiCad schematic (older format))
At the start: 23 parts

Commit message: Updated dac.sch
Other:
- note added: "I2S (Optional)"
- moved on the sheet: J?
Changed lines of the file:
@@
 Wire Wire Line
 	4700 3100 4500 3100
-Text HLabel 2200 4850 0    50   Output ~ 0
+Text HLabel 3350 1750 0    50   Output ~ 0
 DAC_WS
-Text HLabel 2200 5050 0    50   Output ~ 0
+Text HLabel 3350 1950 0    50   Output ~ 0
 DAC_CK
-Text HLabel 2200 5150 0    50   Output ~ 0
+Text HLabel 3350 2050 0    50   Output ~ 0
 DAC_MCK
 $Comp
 L power:GNDD #PWR?
 U 1 1 614A031D
-P 2200 5350
-F 0 "#PWR?" H 2200 5100 50  0001 C CNN
-F 1 "GNDD" H 2204 5195 50  0000 C CNN
-F 2 "" H 2200 5350 50  0001 C CNN
-F 3 "" H 2200 5350 50  0001 C CNN
-	1    2200 5350
+P 3350 2250
+F 0 "#PWR?" H 3350 2000 50  0001 C CNN
+F 1 "GNDD" H 3354 2095 50  0000 C CNN
+F 2 "" H 3350 2250 50  0001 C CNN
+F 3 "" H 3350 2250 50  0001 C CNN
+	1    3350 2250
 	1    0    0    -1
 $EndComp
@@
 L power:+3.3V #PWR?
 U 1 1 614A34C6
-P 2200 4650
-F 0 "#PWR?" H 2200 4500 50  0001 C CNN
-F 1 "+3.3V" H 2215 4823 50  0000 C CNN
-F 2 "" H 2200 4650 50  0001 C CNN
-F 3 "" H 2200 4650 50  0001 C CNN
-	1    2200 4650
+P 3350 1550
+F 0 "#PWR?" H 3350 1400 50  0001 C CNN
+F 1 "+3.3V" H 3365 1723 50  0000 C CNN
+F 2 "" H 3350 1550 50  0001 C CNN
+F 3 "" H 3350 1550 50  0001 C CNN
+	1    3350 1550
 	1    0    0    -1
 $EndComp
@@
 L Connector_Generic:Conn_01x06 J?
 U 1 1 614C038E
-P 2500 4950
-F 0 "J?" H 2580 4942 50  0000 L CNN
-F 1 "Conn_01x06" H 2580 4851 50  0000 L CNN
-F 2 "Connector_PinHeader_2.54mm:PinHeader_1x06_P2.54mm_Vertical" H 2500 4950 50  0001 C CNN
-F 3 "~" H 2500 4950 50  0001 C CNN
-	1    2500 4950
-	1    0    0    -1
-$EndComp
-Wire Wire Line
-	2300 4850 2200 4850
-Wire Wire Line
-	2300 5050 2200 5050
-Wire Wire Line
-	2300 4950 2200 4950
-Wire Wire Line
-	2300 5150 2200 5150
-Wire Wire Line
-	2300 5250 2200 5250
-Wire Wire Line
-	2200 5250 2200 5350
-Wire Wire Line
-	2300 4750 2200 4750
-Wire Wire Line
-	2200 4750 2200 4650
+P 3650 1850
+F 0 "J?" H 3730 1842 50  0000 L CNN
+F 1 "Conn_01x06" H 3730 1751 50  0000 L CNN
+F 2 "Connector_PinHeader_2.54mm:PinHeader_1x06_P2.54mm_Vertical" H 3650 1850 50  0001 C CNN
+F 3 "~" H 3650 1850 50  0001 C CNN
+	1    3650 1850
+	1    0    0    -1
+$EndComp
+Wire Wire Line
+	3450 1750 3350 1750
+Wire Wire Line
+	3450 1950 3350 1950
+Wire Wire Line
+	3450 1850 3350 1850
+Wire Wire Line
+	3450 2050 3350 2050
+Wire Wire Line
+	3450 2150 3350 2150
+Wire Wire Line
+	3350 2150 3350 2250
+Wire Wire Line
+	3450 1650 3350 1650
+Wire Wire Line
+	3350 1650 3350 1550
 $Comp
 L Connector_Generic:Conn_01x03 J?
@@
 Wire Wire Line
 	9950 3450 9950 3650
-Text HLabel 2200 4950 0    50   Output ~ 0
+Text HLabel 3350 1850 0    50   Output ~ 0
 DAC_SD
 $Comp
@@
 Wire Notes Line
 	4750 1850 4750 1250
+Wire Notes Line
+	2800 1250 4300 1250
+Wire Notes Line
+	2800 2550 4300 2550
+Wire Notes Line
+	4300 1250 4300 2550
+Wire Notes Line
+	2800 2550 2800 1250
+Text Notes 2800 1200 0    50   ~ 0
+I2S (Optional)
 $EndSCHEMATC
