File: hardware/sound-20d01mb/dac.sch (KiCad schematic (older format))
At the start: 23 parts

Commit message: PCM5142 I2C Mode
Parts:
- U?: symbol sound-20d01_Library:PCM5142 -> sound-20d01_Library:PCM5142_I2C
Changed lines of the file:
@@
 DAC_SD
 $Comp
-L sound-20d01_Library:PCM5142 U?
+L sound-20d01_Library:PCM5142_I2C U?
 U 1 1 6140DEF6
 P 5500 3350

Commit message: Annotate schematic
Parts:
- gave numbers to parts that had none: 23
