File: hardware/sound-20d01mb/sound-20d01mb.kicad_pcb (KiCad board)
At the start: 2 copper layers, 199.4 x 69.9 mm, 123 parts, among them J1 USB_B, J10 Conn_01x02, J11 Conn_01x03, J12 Conn_01x04, J13 Conn_01x06, J14 Conn_01x03, J2 Conn_01x04, J3 Conn_02x08_Odd_Even, J4 Conn_02x04_Odd_Even, J5 Conn_01x06, J6 Conn_02x10_Odd_Even, J7 Conn_02x10_Odd_Even, J8 Conn_01x02, J9 Conn_01x02, SW1 SW_DIP_x02, U1 USBLC6-2SC6, U2 STM32F446RCTx, U3 PCM5142, U4 TPA3123D2, U5 PC817, U6 PC817, U7 ADP3338AKCZ-3.3RL7, U8 ADP3338AKCZ-3.3RL7, U9 L7805ABD2T-TR, X1 SM7745HEV-12.288M, Y1 32.768kHz, Y2 8MHz

Commit message: Added PWP0024B
Parts:
- U4: footprint Package_SO:HTSSOP-24-1EP_4.4x7.8mm_P0.65mm_EP3.4x7.8mm_Mask2.4x4.68mm_ThermalVias -> sound-20d01mb:PWP0024B
Routing:
- net VCC: track 83.3 -> 93.2 mm
- net GNDA: track 0.00 -> 8.67 mm

Commit message: Updated PCB
Parts:
- moved NT1 5.72 mm to (146.1, 111.1)
Routing:
- net +3V3: track 99.0 -> 390.5 mm, vias 12 -> 15
- net /Amplifier/~SHUTDOWN: track 2.02 -> 48.0 mm, vias 1 -> 2
- net /Amplifier/MUTE: track 2.08 -> 47.0 mm, vias 1 -> 2
- net /Microcontroller Unit/NRST: track 2.96 -> 42.8 mm, vias 0 -> 1
- net PB13: track 0.00 -> 39.5 mm, vias 0 -> 1
- net I2C1_SCL: track 43.1 -> 82.3 mm, vias 0 -> 1
- net I2C1_SDA: track 46.6 -> 81.2 mm, vias 0 -> 1
- net PB15: track 0.00 -> 34.4 mm, vias 0 -> 1
- net PB14: track 0.00 -> 33.9 mm, vias 0 -> 1
- net I2S_OSC_EN: track 0.00 -> 33.2 mm, vias 0 -> 2
- net Net-(JP2-Pad2): track 0.00 -> 28.9 mm, vias 0 -> 1
- net PB5: track 28.0 -> 19.5 mm
- net +5V: track 98.2 -> 105.8 mm
- net GNDD: track 31.3 -> 33.8 mm, vias 18 -> 31
- net GNDA: track 8.67 -> 11.1 mm, vias 23 -> 34
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Other:
- board text added: "BOOT0"
- board text added: "VBAT"
