File: hardware/sound-20d01mb/sound-20d01mb.kicad_pcb (KiCad board)
At the start: 2 copper layers, 199.4 x 69.9 mm, 123 parts, among them J1 USB_B, J10 Conn_01x02, J11 Conn_01x03, J12 Conn_01x04, J13 Conn_01x06, J14 Conn_01x03, J2 Conn_01x04, J3 Conn_02x08_Odd_Even, J4 Conn_02x04_Odd_Even, J5 Conn_01x06, J6 Conn_02x10_Odd_Even, J7 Conn_02x10_Odd_Even, J8 Conn_01x02, J9 Conn_01x02, SW1 SW_DIP_x02, U1 USBLC6-2SC6, U2 STM32F446RCTx, U3 PCM5142, U4 TPA3123D2, U5 PC817, U6 PC817, U7 ADP3338AKCZ-3.3RL7, U8 ADP3338AKCZ-3.3RL7, U9 L7805ABD2T-TR, X1 SM7745HEV-12.288M, Y1 32.768kHz, Y2 8MHz

Commit message: Updated PWP0024B
Routing:
- net GNDA: vias 37 -> 43
Changed lines of the file:
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@@
     (thickness 1.6)
     (drawings 114)
-    (tracks 1261)
+    (tracks 1267)
     (zones 0)
     (modules 123)
@@
       (effects (font (size 1 1) (thickness 0.15)))
     )
-    (pad 25 thru_hole circle (at 0 3) (size 0.8 0.8) (drill 0.4) (layers *.Cu B.Mask)
-      (net 11 GNDA))
-    (pad 25 thru_hole circle (at 1 3) (size 0.8 0.8) (drill 0.4) (layers *.Cu B.Mask)
-      (net 11 GNDA))
-    (pad 25 thru_hole circle (at -1 3) (size 0.8 0.8) (drill 0.4) (layers *.Cu B.Mask)
-      (net 11 GNDA))
-    (pad 25 thru_hole circle (at -1 -3) (size 0.8 0.8) (drill 0.4) (layers *.Cu B.Mask)
-      (net 11 GNDA))
-    (pad 25 thru_hole circle (at 0 -3) (size 0.8 0.8) (drill 0.4) (layers *.Cu B.Mask)
-      (net 11 GNDA))
-    (pad 25 thru_hole circle (at 1 -3) (size 0.8 0.8) (drill 0.4) (layers *.Cu B.Mask)
-      (net 11 GNDA))
     (pad 25 thru_hole circle (at 0 2) (size 0.8 0.8) (drill 0.4) (layers *.Cu *.Mask)
       (net 11 GNDA))
@@
   (segment (start 154.94 115.7875) (end 153.035 115.7875) (width 0.8) (layer F.Cu) (net 10))
   (segment (start 148.59 115.7875) (end 148.59 107.95) (width 1.2) (layer B.Cu) (net 10))
+  (via (at 178.07 93.52) (size 0.8) (drill 0.4) (layers F.Cu B.Cu) (net 11))
   (via (at 189.4475 86.995) (size 0.8) (drill 0.4) (layers F.Cu B.Cu) (net 11))
   (via (at 189.4475 81.915) (size 0.8) (drill 0.4) (layers F.Cu B.Cu) (net 11))
@@
   (via (at 153.035 123.825) (size 0.8) (drill 0.4) (layers F.Cu B.Cu) (net 11))
   (via (at 156.845 123.825) (size 0.8) (drill 0.4) (layers F.Cu B.Cu) (net 11))
+  (via (at 179.07 93.52) (size 0.8) (drill 0.4) (layers F.Cu B.Cu) (net 11))
+  (via (at 180.07 93.52) (size 0.8) (drill 0.4) (layers F.Cu B.Cu) (net 11))
+  (via (at 178.07 99.52) (size 0.8) (drill 0.4) (layers F.Cu B.Cu) (net 11))
+  (via (at 179.07 99.52) (size 0.8) (drill 0.4) (layers F.Cu B.Cu) (net 11))
+  (via (at 180.07 99.52) (size 0.8) (drill 0.4) (layers F.Cu B.Cu) (net 11))
   (segment (start 160.8725 92.71) (end 160.8725 88.265) (width 0.8) (layer F.Cu) (net 12))
   (segment (start 160.8725 92.71) (end 161.925 92.71) (width 0.25) (layer F.Cu) (net 12))
