File: hardware/sound-20d01mb/psu.sch (KiCad schematic (older format))
At the start: 22 parts, among them U7 ADP3338AKCZ-3.3RL7, U8 ADP3338AKCZ-3.3RL7, U9 L7805ABD2T-TR

Commit message: Updated C52 footprint
Parts:
- C52: footprint Capacitor_SMD:CP_Elec_6.3x5.4 -> Capacitor_SMD:CP_Elec_6.3x7.7
Changed lines of the file:
@@
 F 0 "C52" H 7468 4746 50  0000 L CNN
 F 1 "47uF" H 7468 4655 50  0000 L CNN
-F 2 "Capacitor_SMD:CP_Elec_6.3x5.4" H 7388 4550 50  0001 C CNN
+F 2 "Capacitor_SMD:CP_Elec_6.3x7.7" H 7388 4550 50  0001 C CNN
 F 3 "~" H 7350 4700 50  0001 C CNN
 	1    7350 4700

Commit message: Updated text
Other:
- note added: "Place U7 as close\nto the MCU as possible."
- note added: "Place U8 as close\nto the DAC as possible."
- note removed: "Place U? as close\nto the DAC as possible."
- note removed: "Place U? as close\nto the MCU as possible."
Changed lines of the file:
@@
 	6850 3300 6350 3300
 Text Notes 5200 2450 0    50   ~ 0
-Place U? as close\nto the MCU as possible.
+Place U7 as close\nto the MCU as possible.
 $Comp
 L Device:CP C49
@@
 	4450 4950 4950 4950
 Text Notes 5200 4100 0    50   ~ 0
-Place U? as close\nto the DAC as possible.
+Place U8 as close\nto the DAC as possible.
 $Comp
 L Device:LED D4

Commit message: Updated R25
Parts:
- R25: value 330R -> 680R
Changed lines of the file:
@@
 P 7350 3050
 F 0 "R25" H 7420 3096 50  0000 L CNN
-F 1 "330R" H 7420 3005 50  0000 L CNN
+F 1 "680R" H 7420 3005 50  0000 L CNN
 F 2 "Resistor_SMD:R_1206_3216Metric_Pad1.42x1.75mm_HandSolder" V 7280 3050 50  0001 C CNN
 F 3 "~" H 7350 3050 50  0001 C CNN
